File: hardware/nixie-clock/nixie-clock.sch (EAGLE design)
At the start: 0 parts

Commit message: Board design
Parts:
- added C1: 4.7uF, rcl:CPOL-EUE3.5-8
- added C2, C3, C4, C5: 0.1u, rcl:C-EUC0805
- added D1: HER106, diode:DIODE-DO15-12
- added IC1: 74HC595D, 74xx-eu:74HC595D
- added IC2: 74141N, 74xx-eu:74141N
- added JP1: (no value), pinhead:PINHD-1X8
- added L1: 220uH, rcl:L-EU6000-XXX-RC
- added LED1, LED2, LED3, LED4: WS2812B_5050N, WS2812B:WS2812B_5050N
- added N1, N2, N3, N4: IN-14, russian-nixies:IN-14
- added OK1, OK2, OK3, OK4: TIL197, optocoupler:TIL197
- added Q1: IRF840, IRF840:IRF840
- added R1: 330, rcl:R-EU_0207/7
- added R2: 22, rcl:R-EU_0207/7
- added R3: 10K, rcl:R-EU_0207/7
- added R4: 470, rcl:R-EU_0207/7
Connections:
- new net +UB: C1.+, D1.C, R1.2, R3.2
- new net CLK: IC1A.SCK, JP1.4
- new net DIN: IC1A.SER, JP1.3
- new net GND: C1.-, C2.2, C3.2, C4.2, C5.2, IC1A.G, JP1.1, JP1.8, LED1.GND, LED2.GND, LED3.GND, LED4.GND, Q1.S, R1.1, R4.2
- new net LED_IN: JP1.7, LED1.DI
- new net N$1: Q1.G, R2.2
- new net N$10: IC2A.2, N1.3, N2.3, N3.3, N4.3
- new net N$11: IC2A.3, N1.4, N2.4, N3.4, N4.4
- new net N$12: IC2A.4, N1.5, N2.5, N3.5, N4.5
- new net N$13: IC2A.5, N1.6, N2.6, N3.6, N4.6
- new net N$14: IC2A.6, N1.7, N2.7, N3.7, N4.7
- new net N$15: IC2A.7, N1.8, N2.8, N3.8, N4.8
- new net N$16: IC2A.8, N1.9, N2.9, N3.9, N4.9
- new net N$17: IC2A.9, N1.0, N2.0, N3.0, N4.0
- new net N$18: OK1.COL, OK2.COL, OK3.COL, OK4.COL, R3.1
- new net N$19: OK1.C, OK2.C, OK3.C, OK4.C, R4.1
- new net N$2: D1.A, L1.2, Q1.D
- new net N$20: IC1A.QE, OK1.A
- new net N$21: LED1.DO, LED2.DI
- new net N$22: IC1A.QG, OK3.A
- new net N$23: IC1A.QH, OK4.A
- new net N$24: IC1A.QA, IC2A.A
- new net N$25: IC1A.QB, IC2A.B
- new net N$26: IC1A.QC, IC2A.C
- new net N$27: IC1A.QD, IC2A.D
- new net N$28: IC1A.QF, OK2.A
- new net N$29: LED2.DO, LED3.DI
- new net N$30: LED3.DO, LED4.DI
- new net N$8: IC2A.0, N1.1, N2.1, N3.1, N4.1
- new net N$9: IC2A.1, N1.2, N2.2, N3.2, N4.2
- new net N1_ANODE: N1.A, OK1.EMI
- new net N2_ANODE: N2.A, OK2.EMI
- new net N3_ANODE: N3.A, OK3.EMI
- new net N4_ANODE: N4.A, OK4.EMI
- new net PWM: JP1.6, R2.1
- new net RCLK: IC1A.RCK, JP1.5
- new net VCC: C2.1, C3.1, C4.1, C5.1, IC1A.SCL, JP1.2, L1.1, LED1.VDD, LED2.VDD, LED3.VDD, LED4.VDD
